File: Electronics/OpenBinaural_mic_polarizer.sch (KiCad schematic (older format))
At the start: 22 parts

Commit message: Working version of the circuit
Parts:
- removed C?: C, symbol C
- removed P?: Mic_R, symbol CONN_01X02
- removed R? (x3): R, symbol R
- removed R?: 2K2, symbol R
- removed U?: TL072, symbol TL072
- added C?: CP, symbol CP
- added C?: C, symbol C
- added P?: Mic_R, symbol CONN_01X02
- added R?: R, symbol R
- added R?: 2K2, symbol R
- added U?: TL072, symbol TL072
Connections:
- wire segments 42 -> 41
Other:
- moved on the sheet: C?, P?, R?

Commit message: Simplified polarization circuit
Parts:
- removed C?: CP, symbol CP
- removed C?: C, symbol C
- removed P?: Mic_R, symbol CONN_01X02
- removed R? (x3): R, symbol R
- removed R?: 2K2, symbol R
- removed RV?: POT, symbol POT
- removed U? (x3): TL072, symbol TL072
- added C2: 2.2u, symbol C
- added D1: D, symbol D
- added P2: Mic_R, symbol CONN_01X02
- added R2: 2K2, symbol R
- added R3, R5, R6: 2k2, symbol R
- added R8, R9: 170, symbol R
- added SW1: SWITCH_INV, symbol SWITCH_INV
- added unit 2 of U1
- C1: renamed from C?; value C -> 2.2u
- R4: renamed from R?; value R -> 2k2
- R7: renamed from R?; value R -> 1392
- gave numbers to parts that had none: 7
Connections:
- net labels added: VCC
- net labels removed: +9V, GNDREF, VAA
- wire segments 41 -> 27
Other:
- note removed: "Mic voltage generation"
- note removed: "Place near audio op-amp"
- note removed: "Virtual ground generation (unnecessary)"
- moved on the sheet: C3, D2, P3, R4, R7

Commit message: Simplified polarization circuit
Parts:
- removed R3, R5: 2k2, symbol R
- added C4: 100u, symbol CP
- C3: value CP -> 100u
- R8, R9: value 170 -> 200
Connections:
- net labels added: GNDREF
- wire segments 27 -> 28
Other:
- moved on the sheet: C3
Changed lines of the file:
@@
 L CP C3
 U 1 1 55589323
-P 4700 1650
-F 0 "C3" H 4725 1750 50  0000 L CNN
-F 1 "CP" H 4725 1550 50  0000 L CNN
-F 2 "" H 4738 1500 30  0000 C CNN
-F 3 "" H 4700 1650 60  0000 C CNN
-	1    4700 1650
+P 5800 1600
+F 0 "C3" H 5825 1700 50  0000 L CNN
+F 1 "100u" H 5825 1500 50  0000 L CNN
+F 2 "" H 5838 1450 30  0000 C CNN
+F 3 "" H 5800 1600 60  0000 C CNN
+	1    5800 1600
 	1    0    0    -1
 $EndComp
@@
 Wire Wire Line
 	4600 3700 4750 3700
-$Comp
-L GND #PWR7
-U 1 1 5558C9E5
-P 3400 3900
-F 0 "#PWR7" H 3400 3650 50  0001 C CNN
-F 1 "GND" H 3400 3750 50  0000 C CNN
-F 2 "" H 3400 3900 60  0000 C CNN
-F 3 "" H 3400 3900 60  0000 C CNN
-	1    3400 3900
-	1    0    0    -1
-$EndComp
 Text GLabel 4750 3700 2    60   Output ~ 0
 Lout
@@
 	6350 3850 6400 3850
 $Comp
-L GND #PWR11
+L GND #PWR9
 U 1 1 55592C21
 P 4000 4100
-F 0 "#PWR11" H 4000 3850 50  0001 C CNN
+F 0 "#PWR9" H 4000 3850 50  0001 C CNN
 F 1 "GND" H 4000 3950 50  0000 C CNN
 F 2 "" H 4000 4100 60  0000 C CNN
 F 3 "" H 4000 4100 60  0000 C CNN
 	1    4000 4100
-	1    0    0    -1
-$EndComp
-$Comp
-L GND #PWR16
-U 1 1 55592D1E
-P 4700 1800
-F 0 "#PWR16" H 4700 1550 50  0001 C CNN
-F 1 "GND" H 4700 1650 50  0000 C CNN
-F 2 "" H 4700 1800 60  0000 C CNN
-F 3 "" H 4700 1800 60  0000 C CNN
-	1    4700 1800
 	1    0    0    -1
 $EndComp
@@
 $EndComp
 $Comp
-L GND #PWR18
+L GND #PWR14
 U 1 1 55592FB6
 P 5250 2050
-F 0 "#PWR18" H 5250 1800 50  0001 C CNN
+F 0 "#PWR14" H 5250 1800 50  0001 C CNN
 F 1 "GND" H 5250 1900 50  0000 C CNN
 F 2 "" H 5250 2050 60  0000 C CNN
@@
 	1    0    0    -1
 $EndComp
-$Comp
-L R R3
-U 1 1 555931A5
-P 3400 3450
-F 0 "R3" V 3480 3450 50  0000 C CNN
-F 1 "2k2" V 3400 3450 50  0000 C CNN
-F 2 "" V 3330 3450 30  0000 C CNN
-F 3 "" H 3400 3450 30  0000 C CNN
-	1    3400 3450
-	1    0    0    -1
-$EndComp
 Wire Wire Line
 	3300 3600 3600 3600
@@
 P 5750 3900
 F 0 "R9" V 5830 3900 50  0000 C CNN
-F 1 "170" V 5750 3900 50  0000 C CNN
+F 1 "200" V 5750 3900 50  0000 C CNN
 F 2 "" V 5680 3900 30  0000 C CNN
 F 3 "" H 5750 3900 30  0000 C CNN
@@
 P 5750 3600
 F 0 "R8" V 5830 3600 50  0000 C CNN
-F 1 "170" V 5750 3600 50  0000 C CNN
+F 1 "200" V 5750 3600 50  0000 C CNN
 F 2 "" V 5680 3600 30  0000 C CNN
 F 3 "" H 5750 3600 30  0000 C CNN
@@
 $EndComp
 Wire Wire Line
-	6400 3750 5750 3750
-$Comp
-L GND #PWR20
+	5500 3750 6400 3750
+$Comp
+L GND #PWR17
 U 1 1 55593864
 P 5750 4050
-F 0 "#PWR20" H 5750 3800 50  0001 C CNN
+F 0 "#PWR17" H 5750 3800 50  0001 C CNN
 F 1 "GND" H 5750 3900 50  0000 C CNN
 F 2 "" H 5750 4050 60  0000 C CNN
@@
 Wire Wire Line
 	4600 5350 4750 5350
-$Comp
-L GND #PWR9
-U 1 1 55593F66
-P 3400 5550
-F 0 "#PWR9" H 3400 5300 50  0001 C CNN
-F 1 "GND" H 3400 5400 50  0000 C CNN
-F 2 "" H 3400 5550 60  0000 C CNN
-F 3 "" H 3400 5550 60  0000 C CNN
-	1    3400 5550
-	1    0    0    -1
-$EndComp
 Text GLabel 4750 5350 2    60   Output ~ 0
 Rout
 $Comp
-L GND #PWR13
+L GND #PWR11
 U 1 1 55593F6D
 P 4000 5750
-F 0 "#PWR13" H 4000 5500 50  0001 C CNN
+F 0 "#PWR11" H 4000 5500 50  0001 C CNN
 F 1 "GND" H 4000 5600 50  0000 C CNN
 F 2 "" H 4000 5750 60  0000 C CNN
@@
 F 3 "" H 2600 5500 60  0000 C CNN
 	1    2600 5500
-	1    0    0    -1
-$EndComp
-$Comp
-L R R5
-U 1 1 55593F79
-P 3400 5100
-F 0 "R5" V 3480 5100 50  0000 C CNN
-F 1 "2k2" V 3400 5100 50  0000 C CNN
-F 2 "" V 3330 5100 30  0000 C CNN
-F 3 "" H 3400 5100 30  0000 C CNN
-	1    3400 5100
 	1    0    0    -1
 $EndComp
@@
 	3250 1700 3150 1700
 $Comp
-L VCC #PWR14
+L VCC #PWR12
 U 1 1 55595586
 P 4250 1450
-F 0 "#PWR14" H 4250 1300 50  0001 C CNN
+F 0 "#PWR12" H 4250 1300 50  0001 C CNN
 F 1 "VCC" H 4250 1600 50  0000 C CNN
 F 2 "" H 4250 1450 60  0000 C CNN
@@
 $EndComp
 $Comp
-L VCC #PWR17
+L VCC #PWR13
 U 1 1 555956D3
 P 5250 1350
-F 0 "#PWR17" H 5250 1200 50  0001 C CNN
+F 0 "#PWR13" H 5250 1200 50  0001 C CNN
 F 1 "VCC" H 5250 1500 50  0000 C CNN
 F 2 "" H 5250 1350 60  0000 C CNN
@@
 $EndComp
 $Comp
-L VCC #PWR6
-U 1 1 5559584E
-P 3400 3300
-F 0 "#PWR6" H 3400 3150 50  0001 C CNN
-F 1 "VCC" H 3400 3450 50  0000 C CNN
-F 2 "" H 3400 3300 60  0000 C CNN
-F 3 "" H 3400 3300 60  0000 C CNN
-	1    3400 3300
-	1    0    0    -1
-$EndComp
-$Comp
-L VCC #PWR10
+L VCC #PWR8
 U 1 1 55595883
 P 4000 3300
-F 0 "#PWR10" H 4000 3150 50  0001 C CNN
+F 0 "#PWR8" H 4000 3150 50  0001 C CNN
 F 1 "VCC" H 4000 3450 50  0000 C CNN
 F 2 "" H 4000 3300 60  0000 C CNN
@@
 $EndComp
 $Comp
-L VCC #PWR19
+L VCC #PWR16
 U 1 1 555958B8
 P 5750 3450
-F 0 "#PWR19" H 5750 3300 50  0001 C CNN
+F 0 "#PWR16" H 5750 3300 50  0001 C CNN
 F 1 "VCC" H 5750 3600 50  0000 C CNN
 F 2 "" H 5750 3450 60  0000 C CNN
@@
 $EndComp
 $Comp
-L VCC #PWR12
+L VCC #PWR10
 U 1 1 55595980
 P 4000 4950
-F 0 "#PWR12" H 4000 4800 50  0001 C CNN
+F 0 "#PWR10" H 4000 4800 50  0001 C CNN
 F 1 "VCC" H 4000 5100 50  0000 C CNN
 F 2 "" H 4000 4950 60  0000 C CNN
 F 3 "" H 4000 4950 60  0000 C CNN
 	1    4000 4950
-	1    0    0    -1
-$EndComp
-$Comp
-L VCC #PWR8
-U 1 1 55595AB1
-P 3400 4950
-F 0 "#PWR8" H 3400 4800 50  0001 C CNN
-F 1 "VCC" H 3400 5100 50  0000 C CNN
-F 2 "" H 3400 4950 60  0000 C CNN
-F 3 "" H 3400 4950 60  0000 C CNN
-	1    3400 4950
 	1    0    0    -1
 $EndComp
@@
 $EndComp
 $Comp
-L VCC #PWR15
+L VCC #PWR18
 U 1 1 55595BAE
-P 4700 1500
-F 0 "#PWR15" H 4700 1350 50  0001 C CNN
-F 1 "VCC" H 4700 1650 50  0000 C CNN
-F 2 "" H 4700 1500 60  0000 C CNN
-F 3 "" H 4700 1500 60  0000 C CNN
-	1    4700 1500
-	1    0    0    -1
-$EndComp
+P 5800 1450
+F 0 "#PWR18" H 5800 1300 50  0001 C CNN
+F 1 "VCC" H 5800 1600 50  0000 C CNN
+F 2 "" H 5800 1450 60  0000 C CNN
+F 3 "" H 5800 1450 60  0000 C CNN
+	1    5800 1450
+	1    0    0    -1
+$EndComp
+$Comp
+L GNDREF #PWR15
+U 1 1 55593B36
+P 5500 3750
+F 0 "#PWR15" H 5500 3500 50  0001 C CNN
+F 1 "GNDREF" H 5500 3600 50  0000 C CNN
+F 2 "" H 5500 3750 60  0000 C CNN
+F 3 "" H 5500 3750 60  0000 C CNN
+	1    5500 3750
+	1    0    0    -1
+$EndComp
+Connection ~ 5750 3750
+$Comp
+L GNDREF #PWR6
+U 1 1 55593BEF
+P 3400 3900
+F 0 "#PWR6" H 3400 3650 50  0001 C CNN
+F 1 "GNDREF" H 3400 3750 50  0000 C CNN
+F 2 "" H 3400 3900 60  0000 C CNN
+F 3 "" H 3400 3900 60  0000 C CNN
+	1    3400 3900
+	1    0    0    -1
+$EndComp
+$Comp
+L GNDREF #PWR7
+U 1 1 55593C7F
+P 3400 5550
+F 0 "#PWR7" H 3400 5300 50  0001 C CNN
+F 1 "GNDREF" H 3400 5400 50  0000 C CNN
+F 2 "" H 3400 5550 60  0000 C CNN
+F 3 "" H 3400 5550 60  0000 C CNN
+	1    3400 5550
+	1    0    0    -1
+$EndComp
+$Comp
+L CP C4
+U 1 1 5559418C
+P 5800 1900
+F 0 "C4" H 5825 2000 50  0000 L CNN
+F 1 "100u" H 5825 1800 50  0000 L CNN
+F 2 "" H 5838 1750 30  0000 C CNN
+F 3 "" H 5800 1900 60  0000 C CNN
+	1    5800 1900
+	1    0    0    -1
+$EndComp
+$Comp
+L GND #PWR19
+U 1 1 55594A46
+P 5800 2050
+F 0 "#PWR19" H 5800 1800 50  0001 C CNN
+F 1 "GND" H 5800 1900 50  0000 C CNN
+F 2 "" H 5800 2050 60  0000 C CNN
+F 3 "" H 5800 2050 60  0000 C CNN
+	1    5800 2050
+	1    0    0    -1
+$EndComp
+$Comp
+L GNDREF #PWR20
+U 1 1 55594AF2
+P 6100 1750
+F 0 "#PWR20" H 6100 1500 50  0001 C CNN
+F 1 "GNDREF" H 6100 1600 50  0000 C CNN
+F 2 "" H 6100 1750 60  0000 C CNN
+F 3 "" H 6100 1750 60  0000 C CNN
+	1    6100 1750
+	1    0    0    -1
+$EndComp
+Wire Wire Line
+	6100 1750 5800 1750
 $EndSCHEMATC
