File: Electronics/Amplifier/stereo_mic_amplifier.sch (KiCad schematic (older format))
At the start: 19 parts

Commit message: Finished schematic
Parts:
- removed C? (x2): C, symbol C
- removed C? (x3): 2.2uF, symbol CP
- removed P?: mic_R, symbol CONN_01X02
- removed RV?: Dual A100K, symbol DUAL_POT
- removed SW?: switch, symbol SWITCH_INV
- removed U?: TL072, symbol TL072
- added C2, C8, C9: 2.2uF, symbol CP
- added C5: 15pF, symbol C
- added C7: 100nF, symbol C
- added P2: mic_R, symbol CONN_01X02
- added R1, R2, R7: 13.7k, symbol R
- added R3, R4, R8, R9: 100k, symbol R
- added R5, R6: 51, symbol R
- added RV1: Dual A100K, symbol DUAL_POT
- added unit 2 of U1
- C4: renamed from C?; value C -> 15pF
- C6: renamed from C?; value 2.2uF -> 22uF
- D1: renamed from D?; value D -> 1N4001
- gave numbers to parts that had none: 7
Connections:
- net labels added: L_out, R_out, pot_a_L, pot_a_R, pot_b_L, pot_b_R, vgnd
- wire segments 0 -> 24
Other:
- moved on the sheet: C1, C3, C4, C6, D1, D2, P1, P3, P4, U1A

Commit message: Specified footprints
Parts:
- C1, C2, C3, C6, C8, C9: footprint (none) -> Discret:C1V8
- C4, C5, C7: footprint (none) -> Capacitors_ThroughHole:C_Disc_D7.5_P5
- D1: footprint (none) -> Discret:D3
- D2: footprint (none) -> LEDs:LED-5MM
- P1, P2, P3: footprint (none) -> Pin_Headers:Pin_Header_Straight_1x02
- P4: footprint (none) -> Pin_Headers:Pin_Header_Straight_1x03
- R1, R2, R3, R4, R5, R6, R7, R8, R9: footprint (none) -> Resistors_ThroughHole:Resistor_Horizontal_RM10mm
- RV1: footprint (none) -> Potentiometers:Potentiometer_Alps-RK163-double_15mm
- U1: footprint (none) -> Sockets_DIP:DIP-8__300_ELL
Changed lines of the file:
@@
 LIBS:memory
 LIBS:xilinx
+LIBS:special
 LIBS:microcontrollers
 LIBS:dsp
@@
 F 0 "U1" H 2800 3700 60  0000 L CNN
 F 1 "TL072" H 2800 3250 60  0000 L CNN
-F 2 "" H 2850 3500 60  0000 C CNN
+F 2 "Sockets_DIP:DIP-8__300_ELL" H 2850 3500 60  0001 C CNN
 F 3 "" H 2850 3500 60  0000 C CNN
 	1    2850 3500
@@
 F 0 "D2" V 3900 1050 50  0000 C CNN
 F 1 "LED" V 3800 1050 50  0000 C CNN
-F 2 "" H 3850 1200 60  0000 C CNN
+F 2 "LEDs:LED-5MM" H 3850 1200 60  0001 C CNN
 F 3 "" H 3850 1200 60  0000 C CNN
 	1    3850 1200
@@
 F 0 "P3" H 2100 1300 50  0000 C CNN
 F 1 "batt" H 2100 1000 50  0000 C CNN
-F 2 "" H 2100 1150 60  0000 C CNN
+F 2 "Pin_Headers:Pin_Header_Straight_1x02" H 2100 1150 60  0001 C CNN
 F 3 "" H 2100 1150 60  0000 C CNN
 	1    2100 1150
@@
 F 0 "D1" V 2450 1350 50  0000 C CNN
 F 1 "1N4001" V 2550 1450 50  0000 C CNN
-F 2 "" H 2500 1250 60  0000 C CNN
+F 2 "Discret:D3" H 2500 1250 60  0001 C CNN
 F 3 "" H 2500 1250 60  0000 C CNN
 	1    2500 1250
@@
 F 0 "C4" V 2600 4350 50  0000 L CNN
 F 1 "15pF" V 2900 4350 50  0000 L CNN
-F 2 "" H 2788 4250 30  0000 C CNN
+F 2 "Capacitors_ThroughHole:C_Disc_D7.5_P5" H 2788 4250 30  0001 C CNN
 F 3 "" H 2750 4400 60  0000 C CNN
 	1    2750 4400
@@
 F 0 "C1" V 1800 3550 50  0000 L CNN
 F 1 "2.2uF" V 2100 3550 50  0000 L CNN
-F 2 "" H 1988 3450 30  0000 C CNN
+F 2 "Discret:C1V8" H 1988 3450 30  0001 C CNN
 F 3 "" H 1950 3600 60  0000 C CNN
 	1    1950 3600
@@
 F 0 "C3" H 2425 2450 50  0000 L CNN
 F 1 "2.2uF" H 2425 2250 50  0000 L CNN
-F 2 "" H 2438 2200 30  0000 C CNN
+F 2 "Discret:C1V8" H 2438 2200 30  0001 C CNN
 F 3 "" H 2400 2350 60  0000 C CNN
 	1    2400 2350
@@
 F 0 "C6" H 3325 1250 50  0000 L CNN
 F 1 "22uF" H 3325 1050 50  0000 L CNN
-F 2 "" H 3338 1000 30  0000 C CNN
+F 2 "Discret:C1V8" H 3338 1000 30  0001 C CNN
 F 3 "" H 3300 1150 60  0000 C CNN
 	1    3300 1150
@@
 F 0 "P1" H 1300 3800 50  0000 C CNN
 F 1 "mic_L" H 1250 3500 50  0000 C CNN
-F 2 "" H 1300 3650 60  0000 C CNN
+F 2 "Pin_Headers:Pin_Header_Straight_1x02" H 1300 3650 60  0001 C CNN
 F 3 "" H 1300 3650 60  0000 C CNN
 	1    1300 3650
@@
 F 0 "P4" H 4500 2450 50  0000 C CNN
 F 1 "CONN_01X03" V 4600 2250 50  0000 C CNN
-F 2 "" H 4500 2250 60  0000 C CNN
+F 2 "Pin_Headers:Pin_Header_Straight_1x03" H 4500 2250 60  0001 C CNN
 F 3 "" H 4500 2250 60  0000 C CNN
 	1    4500 2250
@@
 F 0 "C7" H 3325 2150 50  0000 L CNN
 F 1 "100nF" H 3325 1950 50  0000 L CNN
-F 2 "" H 3338 1900 30  0000 C CNN
+F 2 "Capacitors_ThroughHole:C_Disc_D7.5_P5" H 3338 1900 30  0001 C CNN
 F 3 "" H 3300 2050 60  0000 C CNN
 	1    3300 2050
@@
 F 0 "R3" H 2200 2100 50  0000 C CNN
 F 1 "100k" H 2250 2000 50  0000 C CNN
-F 2 "" V 2030 2050 30  0000 C CNN
+F 2 "Resistors_ThroughHole:Resistor_Horizontal_RM10mm" V 2030 2050 30  0001 C CNN
 F 3 "" H 2100 2050 30  0000 C CNN
 	1    2100 2050
@@
 F 0 "R1" H 1750 3350 50  0000 C CNN
 F 1 "13.7k" H 1800 3250 50  0000 C CNN
-F 2 "" V 1580 3300 30  0000 C CNN
+F 2 "Resistors_ThroughHole:Resistor_Horizontal_RM10mm" V 1580 3300 30  0001 C CNN
 F 3 "" H 1650 3300 30  0000 C CNN
 	1    1650 3300
@@
 F 0 "R4" H 2200 2400 50  0000 C CNN
 F 1 "100k" H 2250 2250 50  0000 C CNN
-F 2 "" V 2030 2350 30  0000 C CNN
+F 2 "Resistors_ThroughHole:Resistor_Horizontal_RM10mm" V 2030 2350 30  0001 C CNN
 F 3 "" H 2100 2350 30  0000 C CNN
 	1    2100 2350
@@
 F 0 "R5" V 3400 3450 50  0000 C CNN
 F 1 "51" V 3600 3500 50  0000 C CNN
-F 2 "" V 3430 3500 30  0000 C CNN
+F 2 "Resistors_ThroughHole:Resistor_Horizontal_RM10mm" V 3430 3500 30  0001 C CNN
 F 3 "" H 3500 3500 30  0000 C CNN
 	1    3500 3500
@@
 F 0 "C8" V 3950 3450 50  0000 L CNN
 F 1 "2.2uF" V 3650 3350 50  0000 L CNN
-F 2 "" H 3838 3350 30  0000 C CNN
+F 2 "Discret:C1V8" H 3838 3350 30  0001 C CNN
 F 3 "" H 3800 3500 60  0000 C CNN
 	1    3800 3500
@@
 F 0 "RV1" H 5860 5260 50  0000 C CNN
 F 1 "Dual A100K" H 5990 4650 50  0000 C CNN
-F 2 "" H 5700 4950 60  0000 C CNN
+F 2 "Potentiometers:Potentiometer_Alps-RK163-double_15mm" H 5700 4950 60  0001 C CNN
 F 3 "" H 5700 4950 60  0000 C CNN
 	1    5700 4950
@@
 F 0 "R8" H 4250 3700 50  0000 C CNN
 F 1 "100k" H 4300 3600 50  0000 C CNN
-F 2 "" V 4080 3650 30  0000 C CNN
+F 2 "Resistors_ThroughHole:Resistor_Horizontal_RM10mm" V 4080 3650 30  0001 C CNN
 F 3 "" H 4150 3650 30  0000 C CNN
 	1    4150 3650
@@
 F 0 "R7" H 3950 1600 50  0000 C CNN
 F 1 "13.7k" H 4000 1500 50  0000 C CNN
-F 2 "" V 3780 1550 30  0000 C CNN
+F 2 "Resistors_ThroughHole:Resistor_Horizontal_RM10mm" V 3780 1550 30  0001 C CNN
 F 3 "" H 3850 1550 30  0000 C CNN
 	1    3850 1550
@@
 F 0 "U1" H 2800 5650 60  0000 L CNN
 F 1 "TL072" H 2800 5200 60  0000 L CNN
-F 2 "" H 2850 5450 60  0000 C CNN
+F 2 "Sockets_DIP:DIP-8__300_ELL" H 2850 5450 60  0001 C CNN
 F 3 "" H 2850 5450 60  0000 C CNN
 	2    2850 5450
@@
 F 0 "C5" V 2600 6300 50  0000 L CNN
 F 1 "15pF" V 2900 6300 50  0000 L CNN
-F 2 "" H 2788 6200 30  0000 C CNN
+F 2 "Capacitors_ThroughHole:C_Disc_D7.5_P5" H 2788 6200 30  0001 C CNN
 F 3 "" H 2750 6350 60  0000 C CNN
 	1    2750 6350
@@
 F 0 "C2" V 1800 5500 50  0000 L CNN
 F 1 "2.2uF" V 2100 5500 50  0000 L CNN
-F 2 "" H 1988 5400 30  0000 C CNN
+F 2 "Discret:C1V8" H 1988 5400 30  0001 C CNN
 F 3 "" H 1950 5550 60  0000 C CNN
 	1    1950 5550
@@
 F 0 "P2" H 1300 5750 50  0000 C CNN
 F 1 "mic_R" H 1250 5450 50  0000 C CNN
-F 2 "" H 1300 5600 60  0000 C CNN
+F 2 "Pin_Headers:Pin_Header_Straight_1x02" H 1300 5600 60  0001 C CNN
 F 3 "" H 1300 5600 60  0000 C CNN
 	1    1300 5600
@@
 F 0 "R2" H 1750 5300 50  0000 C CNN
 F 1 "13.7k" H 1800 5200 50  0000 C CNN
-F 2 "" V 1580 5250 30  0000 C CNN
+F 2 "Resistors_ThroughHole:Resistor_Horizontal_RM10mm" V 1580 5250 30  0001 C CNN
 F 3 "" H 1650 5250 30  0000 C CNN
 	1    1650 5250
@@
 F 0 "R6" V 3400 5400 50  0000 C CNN
 F 1 "51" V 3600 5450 50  0000 C CNN
-F 2 "" V 3430 5450 30  0000 C CNN
+F 2 "Resistors_ThroughHole:Resistor_Horizontal_RM10mm" V 3430 5450 30  0001 C CNN
 F 3 "" H 3500 5450 30  0000 C CNN
 	1    3500 5450
@@
 F 0 "C9" V 3950 5400 50  0000 L CNN
 F 1 "2.2uF" V 3650 5300 50  0000 L CNN
-F 2 "" H 3838 5300 30  0000 C CNN
+F 2 "Discret:C1V8" H 3838 5300 30  0001 C CNN
 F 3 "" H 3800 5450 60  0000 C CNN
 	1    3800 5450
@@
 F 0 "R9" H 4250 5650 50  0000 C CNN
 F 1 "100k" H 4300 5550 50  0000 C CNN
-F 2 "" V 4080 5600 30  0000 C CNN
+F 2 "Resistors_ThroughHole:Resistor_Horizontal_RM10mm" V 4080 5600 30  0001 C CNN
 F 3 "" H 4150 5600 30  0000 C CNN
 	1    4150 5600

Commit message: Fixed dual potentiometer pins
Connections:
- net GND: now also D1.2 (K), P3.1 (P1)
Other:
- moved on the sheet: C8, C9, R3, R5, R6, R8, R9
Changed lines of the file:
@@
 L R R3
 U 1 1 55799796
-P 2100 2050
-F 0 "R3" H 2200 2100 50  0000 C CNN
-F 1 "100k" H 2250 2000 50  0000 C CNN
-F 2 "Resistors_ThroughHole:Resistor_Horizontal_RM10mm" V 2030 2050 30  0001 C CNN
-F 3 "" H 2100 2050 30  0000 C CNN
-	1    2100 2050
-	1    0    0    -1
-$EndComp
-Wire Wire Line
-	2100 2200 2600 2200
+P 2100 2000
+F 0 "R3" H 2200 2050 50  0000 C CNN
+F 1 "100k" H 2250 1950 50  0000 C CNN
+F 2 "Resistors_ThroughHole:Resistor_Horizontal_RM10mm" V 2030 2000 30  0001 C CNN
+F 3 "" H 2100 2000 30  0000 C CNN
+	1    2100 2000
+	1    0    0    -1
+$EndComp
 $Comp
 L +9V #PWR05
 U 1 1 55799832
-P 2100 1900
-F 0 "#PWR05" H 2100 1750 50  0001 C CNN
-F 1 "+9V" H 2100 2040 50  0000 C CNN
-F 2 "" H 2100 1900 60  0000 C CNN
-F 3 "" H 2100 1900 60  0000 C CNN
-	1    2100 1900
+P 2100 1850
+F 0 "#PWR05" H 2100 1700 50  0001 C CNN
+F 1 "+9V" H 2100 1990 50  0000 C CNN
+F 2 "" H 2100 1850 60  0000 C CNN
+F 3 "" H 2100 1850 60  0000 C CNN
+	1    2100 1850
 	1    0    0    -1
 $EndComp
@@
 L GND #PWR06
 U 1 1 55799945
-P 2100 2500
-F 0 "#PWR06" H 2100 2250 50  0001 C CNN
-F 1 "GND" H 2100 2350 50  0000 C CNN
-F 2 "" H 2100 2500 60  0000 C CNN
-F 3 "" H 2100 2500 60  0000 C CNN
-	1    2100 2500
-	1    0    0    -1
-$EndComp
-Wire Wire Line
-	2400 2500 2100 2500
-Connection ~ 2400 2200
+P 2100 2550
+F 0 "#PWR06" H 2100 2300 50  0001 C CNN
+F 1 "GND" H 2100 2400 50  0000 C CNN
+F 2 "" H 2100 2550 60  0000 C CNN
+F 3 "" H 2100 2550 60  0000 C CNN
+	1    2100 2550
+	1    0    0    -1
+$EndComp
 Text GLabel 2600 2200 2    60   Output ~ 0
 vgnd
@@
 	1    0    0    -1
 $EndComp
-Wire Wire Line
-	1500 3600 1800 3600
-Wire Wire Line
-	1650 3450 1650 3600
-Connection ~ 1650 3600
 $Comp
 L GND #PWR07
@@
 L R R5
 U 1 1 5579BB59
-P 3500 3500
-F 0 "R5" V 3400 3450 50  0000 C CNN
-F 1 "51" V 3600 3500 50  0000 C CNN
-F 2 "Resistors_ThroughHole:Resistor_Horizontal_RM10mm" V 3430 3500 30  0001 C CNN
-F 3 "" H 3500 3500 30  0000 C CNN
-	1    3500 3500
+P 3550 3500
+F 0 "R5" V 3450 3450 50  0000 C CNN
+F 1 "51" V 3650 3500 50  0000 C CNN
+F 2 "Resistors_ThroughHole:Resistor_Horizontal_RM10mm" V 3480 3500 30  0001 C CNN
+F 3 "" H 3550 3500 30  0000 C CNN
+	1    3550 3500
 	0    1    1    0
 $EndComp
@@
 L CP C8
 U 1 1 5579BDA4
-P 3800 3500
-F 0 "C8" V 3950 3450 50  0000 L CNN
-F 1 "2.2uF" V 3650 3350 50  0000 L CNN
-F 2 "Discret:C1V8" H 3838 3350 30  0001 C CNN
-F 3 "" H 3800 3500 60  0000 C CNN
-	1    3800 3500
+P 3850 3500
+F 0 "C8" V 4000 3450 50  0000 L CNN
+F 1 "2.2uF" V 3700 3350 50  0000 L CNN
+F 2 "Discret:C1V8" H 3888 3350 30  0001 C CNN
+F 3 "" H 3850 3500 60  0000 C CNN
+	1    3850 3500
 	0    -1   -1   0
 $EndComp
-Wire Wire Line
-	2350 3600 2100 3600
 $Comp
 L DUAL_POT RV1
@@
 	1    0    0    -1
 $EndComp
-Wire Wire Line
-	2350 3600 2350 4700
-Wire Wire Line
-	2350 4400 2600 4400
-Wire Wire Line
-	2900 4400 3350 4400
-Wire Wire Line
-	3350 3500 3350 4700
 Text GLabel 2350 4700 2    60   BiDi ~ 0
 pot_a_L
 Text GLabel 3350 4700 2    60   BiDi ~ 0
 pot_b_L
-Connection ~ 3350 4400
-Connection ~ 2350 4400
 Text GLabel 5550 4650 0    60   BiDi ~ 0
 pot_a_L
 Text GLabel 6000 4750 2    60   BiDi ~ 0
 pot_b_L
-Text GLabel 4350 3500 2    60   Output ~ 0
+Text GLabel 4400 3500 2    60   Output ~ 0
 L_out
 Text GLabel 4250 2150 0    60   Input ~ 0
@@
 Text GLabel 4250 2350 0    60   Input ~ 0
 R_out
-Wire Wire Line
-	4300 2250 3800 2250
-Wire Wire Line
-	4300 2350 4250 2350
-Wire Wire Line
-	4300 2150 4250 2150
 $Comp
 L R R8
 U 1 1 5579F1EE
-P 4150 3650
-F 0 "R8" H 4250 3700 50  0000 C CNN
-F 1 "100k" H 4300 3600 50  0000 C CNN
-F 2 "Resistors_ThroughHole:Resistor_Horizontal_RM10mm" V 4080 3650 30  0001 C CNN
-F 3 "" H 4150 3650 30  0000 C CNN
-	1    4150 3650
-	1    0    0    -1
-$EndComp
-Wire Wire Line
-	3950 3500 4350 3500
-Connection ~ 4150 3500
+P 4200 3650
+F 0 "R8" H 4300 3700 50  0000 C CNN
+F 1 "100k" H 4350 3600 50  0000 C CNN
+F 2 "Resistors_ThroughHole:Resistor_Horizontal_RM10mm" V 4130 3650 30  0001 C CNN
+F 3 "" H 4200 3650 30  0000 C CNN
+	1    4200 3650
+	1    0    0    -1
+$EndComp
 $Comp
 L GND #PWR09
 U 1 1 5579F3B2
-P 4150 3800
-F 0 "#PWR09" H 4150 3550 50  0001 C CNN
-F 1 "GND" H 4150 3650 50  0000 C CNN
-F 2 "" H 4150 3800 60  0000 C CNN
-F 3 "" H 4150 3800 60  0000 C CNN
-	1    4150 3800
+P 4200 3800
+F 0 "#PWR09" H 4200 3550 50  0001 C CNN
+F 1 "GND" H 4200 3650 50  0000 C CNN
+F 2 "" H 4200 3800 60  0000 C CNN
+F 3 "" H 4200 3800 60  0000 C CNN
+	1    4200 3800
 	1    0    0    -1
 $EndComp
@@
 L +9V #PWR011
 U 1 1 557A0042
-P 2300 1100
-F 0 "#PWR011" H 2300 950 50  0001 C CNN
-F 1 "+9V" H 2300 1240 50  0000 C CNN
-F 2 "" H 2300 1100 60  0000 C CNN
-F 3 "" H 2300 1100 60  0000 C CNN
-	1    2300 1100
+P 2400 1000
+F 0 "#PWR011" H 2400 850 50  0001 C CNN
+F 1 "+9V" H 2400 1140 50  0000 C CNN
+F 2 "" H 2400 1000 60  0000 C CNN
+F 3 "" H 2400 1000 60  0000 C CNN
+	1    2400 1000
 	1    0    0    -1
 $EndComp
@@
 	1    0    0    -1
 $EndComp
-Wire Wire Line
-	2500 1100 2300 1100
 $Comp
 L +9V #PWR016
@@
 	1    0    0    -1
 $EndComp
-Wire Wire Line
-	1500 5550 1800 5550
-Wire Wire Line
-	1650 5400 1650 5550
-Connection ~ 1650 5550
 $Comp
 L GND #PWR019
@@
 L R R6
 U 1 1 557A3231
-P 3500 5450
-F 0 "R6" V 3400 5400 50  0000 C CNN
-F 1 "51" V 3600 5450 50  0000 C CNN
-F 2 "Resistors_ThroughHole:Resistor_Horizontal_RM10mm" V 3430 5450 30  0001 C CNN
-F 3 "" H 3500 5450 30  0000 C CNN
-	1    3500 5450
+P 3550 5450
+F 0 "R6" V 3450 5400 50  0000 C CNN
+F 1 "51" V 3650 5450 50  0000 C CNN
+F 2 "Resistors_ThroughHole:Resistor_Horizontal_RM10mm" V 3480 5450 30  0001 C CNN
+F 3 "" H 3550 5450 30  0000 C CNN
+	1    3550 5450
 	0    1    1    0
 $EndComp
@@
 L CP C9
 U 1 1 557A3237
-P 3800 5450
-F 0 "C9" V 3950 5400 50  0000 L CNN
-F 1 "2.2uF" V 3650 5300 50  0000 L CNN
-F 2 "Discret:C1V8" H 3838 5300 30  0001 C CNN
-F 3 "" H 3800 5450 60  0000 C CNN
-	1    3800 5450
+P 3850 5450
+F 0 "C9" V 4000 5400 50  0000 L CNN
+F 1 "2.2uF" V 3700 5300 50  0000 L CNN
+F 2 "Discret:C1V8" H 3888 5300 30  0001 C CNN
+F 3 "" H 3850 5450 60  0000 C CNN
+	1    3850 5450
 	0    -1   -1   0
 $EndComp
-Wire Wire Line
-	2350 5550 2100 5550
-Wire Wire Line
-	2350 5550 2350 6650
-Wire Wire Line
-	2350 6350 2600 6350
-Wire Wire Line
-	2900 6350 3350 6350
-Wire Wire Line
-	3350 5450 3350 6650
 Text GLabel 2350 6650 2    60   BiDi ~ 0
 pot_a_R
 Text GLabel 3350 6650 2    60   BiDi ~ 0
 pot_b_R
-Connection ~ 3350 6350
-Connection ~ 2350 6350
-Text GLabel 4350 5450 2    60   Output ~ 0
+Text GLabel 4400 5450 2    60   Output ~ 0
 R_out
 $Comp
 L R R9
 U 1 1 557A3247
-P 4150 5600
-F 0 "R9" H 4250 5650 50  0000 C CNN
-F 1 "100k" H 4300 5550 50  0000 C CNN
-F 2 "Resistors_ThroughHole:Resistor_Horizontal_RM10mm" V 4080 5600 30  0001 C CNN
-F 3 "" H 4150 5600 30  0000 C CNN
-	1    4150 5600
-	1    0    0    -1
-$EndComp
-Wire Wire Line
-	3950 5450 4350 5450
-Connection ~ 4150 5450
+P 4200 5600
+F 0 "R9" H 4300 5650 50  0000 C CNN
+F 1 "100k" H 4350 5550 50  0000 C CNN
+F 2 "Resistors_ThroughHole:Resistor_Horizontal_RM10mm" V 4130 5600 30  0001 C CNN
+F 3 "" H 4200 5600 30  0000 C CNN
+	1    4200 5600
+	1    0    0    -1
+$EndComp
 $Comp
 L GND #PWR020
 U 1 1 557A324F
-P 4150 5750
-F 0 "#PWR020" H 4150 5500 50  0001 C CNN
-F 1 "GND" H 4150 5600 50  0000 C CNN
-F 2 "" H 4150 5750 60  0000 C CNN
-F 3 "" H 4150 5750 60  0000 C CNN
-	1    4150 5750
+P 4200 5750
+F 0 "#PWR020" H 4200 5500 50  0001 C CNN
+F 1 "GND" H 4200 5600 50  0000 C CNN
+F 2 "" H 4200 5750 60  0000 C CNN
+F 3 "" H 4200 5750 60  0000 C CNN
+	1    4200 5750
 	1    0    0    -1
 $EndComp
@@
 pot_b_R
 Wire Wire Line
-	2500 1400 2300 1400
-Wire Wire Line
-	2300 1400 2300 1200
+	1500 3600 1800 3600
+Wire Wire Line
+	1650 3450 1650 3600
+Connection ~ 1650 3600
+Wire Wire Line
+	2350 3600 2100 3600
+Wire Wire Line
+	2350 3600 2350 4700
+Wire Wire Line
+	2350 4400 2600 4400
+Connection ~ 2350 4400
+Wire Wire Line
+	4300 2250 3800 2250
+Wire Wire Line
+	4300 2350 4250 2350
+Wire Wire Line
+	4300 2150 4250 2150
+Wire Wire Line
+	4000 3500 4400 3500
+Connection ~ 4200 3500
+Wire Wire Line
+	1500 5550 1800 5550
+Wire Wire Line
+	1650 5400 1650 5550
+Connection ~ 1650 5550
+Wire Wire Line
+	2350 5550 2100 5550
+Wire Wire Line
+	2350 5550 2350 6650
+Wire Wire Line
+	2350 6350 2600 6350
+Connection ~ 2350 6350
+Wire Wire Line
+	4000 5450 4400 5450
+Connection ~ 4200 5450
+Wire Wire Line
+	2300 1400 2500 1400
+Wire Wire Line
+	2300 1200 2300 1400
+Connection ~ 2400 1400
+Wire Wire Line
+	2300 1100 2500 1100
+Wire Wire Line
+	2400 1000 2400 1100
+Connection ~ 2400 1100
+Wire Wire Line
+	2400 2500 2100 2500
+Wire Wire Line
+	2100 2500 2100 2550
+Wire Wire Line
+	2100 2200 2100 2150
+Wire Wire Line
+	2100 2200 2600 2200
+Connection ~ 2400 2200
+Wire Wire Line
+	3400 3500 3350 3500
+Wire Wire Line
+	3350 3500 3350 4700
+Wire Wire Line
+	2900 4400 3350 4400
+Connection ~ 3350 4400
+Wire Wire Line
+	3350 6650 3350 5450
+Wire Wire Line
+	3350 5450 3400 5450
+Wire Wire Line
+	2900 6350 3350 6350
+Connection ~ 3350 6350
 $EndSCHEMATC

Commit message: Work on the layout
Parts:
- removed RV1: Dual A100K, Potentiometers:Potentiometer_Alps-RK163-double_15mm, symbol DUAL_POT
- added RV1: DUAL_POT_OK, Potentiometers:Potentiometer_Alps-RK163-double_15mm, symbol DUAL_POT_OK
Connections:
- net +9V: now also R7.1; no longer D2.2 (K)
- net GND: now also D2.1 (A); no longer R7.2
- net pot_a_L: now also RV1.13
- net pot_a_R: now also RV1.23
- net pot_b_L: now also RV1.12
- net pot_b_R: now also RV1.22
- new net: D2.2 (K), R7.2
Other:
- moved on the sheet: D2, R7
Changed lines of the file:
@@
 LIBS:contrib
 LIBS:valves
-LIBS:stereo_mic_amplifier-cache
+LIBS:mic_amp
 EELAYER 25 0
 EELAYER END
@@
 L LED D2
 U 1 1 5576C5E6
-P 3850 1200
-F 0 "D2" V 3900 1050 50  0000 C CNN
-F 1 "LED" V 3800 1050 50  0000 C CNN
-F 2 "LEDs:LED-5MM" H 3850 1200 60  0001 C CNN
-F 3 "" H 3850 1200 60  0000 C CNN
-	1    3850 1200
+P 3850 1500
+F 0 "D2" V 3900 1350 50  0000 C CNN
+F 1 "LED" V 3800 1350 50  0000 C CNN
+F 2 "LEDs:LED-5MM" H 3850 1500 60  0001 C CNN
+F 3 "" H 3850 1500 60  0000 C CNN
+	1    3850 1500
 	0    -1   -1   0
 $EndComp
@@
 	0    -1   -1   0
 $EndComp
-$Comp
-L DUAL_POT RV1
-U 1 1 5579D759
-P 5700 4950
-F 0 "RV1" H 5860 5260 50  0000 C CNN
-F 1 "Dual A100K" H 5990 4650 50  0000 C CNN
-F 2 "Potentiometers:Potentiometer_Alps-RK163-double_15mm" H 5700 4950 60  0001 C CNN
-F 3 "" H 5700 4950 60  0000 C CNN
-	1    5700 4950
-	1    0    0    -1
-$EndComp
 Text GLabel 2350 4700 2    60   BiDi ~ 0
 pot_a_L
 Text GLabel 3350 4700 2    60   BiDi ~ 0
 pot_b_L
-Text GLabel 5550 4650 0    60   BiDi ~ 0
+Text GLabel 5550 4850 0    60   BiDi ~ 0
 pot_a_L
 Text GLabel 6000 4750 2    60   BiDi ~ 0
@@
 L R R7
 U 1 1 557A0E47
-P 3850 1550
-F 0 "R7" H 3950 1600 50  0000 C CNN
-F 1 "13.7k" H 4000 1500 50  0000 C CNN
-F 2 "Resistors_ThroughHole:Resistor_Horizontal_RM10mm" V 3780 1550 30  0001 C CNN
-F 3 "" H 3850 1550 30  0000 C CNN
-	1    3850 1550
+P 3850 1150
+F 0 "R7" H 3950 1200 50  0000 C CNN
+F 1 "13.7k" H 4000 1100 50  0000 C CNN
+F 2 "Resistors_ThroughHole:Resistor_Horizontal_RM10mm" V 3780 1150 30  0001 C CNN
+F 3 "" H 3850 1150 30  0000 C CNN
+	1    3850 1150
 	1    0    0    -1
 $EndComp
@@
 	1    0    0    -1
 $EndComp
-Text GLabel 5550 5050 0    60   BiDi ~ 0
+Text GLabel 5550 5250 0    60   BiDi ~ 0
 pot_a_R
 Text GLabel 6000 5150 2    60   BiDi ~ 0
@@
 	2900 6350 3350 6350
 Connection ~ 3350 6350
+$Comp
+L DUAL_POT_OK RV1
+U 1 1 557B37A4
+P 5700 4950
+F 0 "RV1" H 5860 5260 50  0000 C CNN
+F 1 "DUAL_POT_OK" H 5990 4650 50  0000 C CNN
+F 2 "Potentiometers:Potentiometer_Alps-RK163-double_15mm" H 5700 4950 60  0001 C CNN
+F 3 "" H 5700 4950 60  0000 C CNN
+	1    5700 4950
+	1    0    0    -1
+$EndComp
 $EndSCHEMATC

Commit message: Layout progress
Parts:
- R5, R6, R8, R9: footprint Resistors_ThroughHole:Resistor_Horizontal_RM10mm -> Resistors_ThroughHole:Resistor_Vertical_RM5mm
Connections:
- net pot_b_L: now also R5.1; no longer R5.2
- net at C8.1: now also R5.2; no longer R5.1
Changed lines of the file:
@@
 LIBS:valves
 LIBS:mic_amp
+LIBS:stereo_mic_amplifier-cache
 EELAYER 25 0
 EELAYER END
@@
 F 0 "R5" V 3450 3450 50  0000 C CNN
 F 1 "51" V 3650 3500 50  0000 C CNN
-F 2 "Resistors_ThroughHole:Resistor_Horizontal_RM10mm" V 3480 3500 30  0001 C CNN
+F 2 "Resistors_ThroughHole:Resistor_Vertical_RM5mm" V 3480 3500 30  0001 C CNN
 F 3 "" H 3550 3500 30  0000 C CNN
 	1    3550 3500
-	0    1    1    0
+	0    -1   -1   0
 $EndComp
 $Comp
@@
 F 0 "R8" H 4300 3700 50  0000 C CNN
 F 1 "100k" H 4350 3600 50  0000 C CNN
-F 2 "Resistors_ThroughHole:Resistor_Horizontal_RM10mm" V 4130 3650 30  0001 C CNN
+F 2 "Resistors_ThroughHole:Resistor_Vertical_RM5mm" V 4130 3650 30  0001 C CNN
 F 3 "" H 4200 3650 30  0000 C CNN
 	1    4200 3650
@@
 F 0 "R6" V 3450 5400 50  0000 C CNN
 F 1 "51" V 3650 5450 50  0000 C CNN
-F 2 "Resistors_ThroughHole:Resistor_Horizontal_RM10mm" V 3480 5450 30  0001 C CNN
+F 2 "Resistors_ThroughHole:Resistor_Vertical_RM5mm" V 3480 5450 30  0001 C CNN
 F 3 "" H 3550 5450 30  0000 C CNN
 	1    3550 5450
@@
 F 0 "R9" H 4300 5650 50  0000 C CNN
 F 1 "100k" H 4350 5550 50  0000 C CNN
-F 2 "Resistors_ThroughHole:Resistor_Horizontal_RM10mm" V 4130 5600 30  0001 C CNN
+F 2 "Resistors_ThroughHole:Resistor_Vertical_RM5mm" V 4130 5600 30  0001 C CNN
 F 3 "" H 4200 5600 30  0000 C CNN
 	1    4200 5600
