File: Electronics/Amplifier/stereo_mic_amplifier.kicad_pcb (KiCad board)
At the start: 2 copper layers, 34.2 x 45.3 mm, 26 parts, among them P1 mic_L, P2 mic_R, P3 batt, P4 CONN_01X03, U1 TL072

Commit message: Finished layout
Parts:
- moved R5 25.0 mm to (79.5, 128.1)
- moved R9 23.7 mm to (104.4, 128.4), turned to 270 degrees
- moved R8 3.22 mm to (83.3, 128.3), turned to 90 degrees
- moved C8 0.46 mm to (90.8, 128.9), turned to 270 degrees
- moved C9 0.13 mm to (97.0, 125.1)
Routing:
- net GND: track 111.8 -> 136.1 mm
- net pot_b_L: track 52.0 -> 72.3 mm
- net R_out: track 0.00 -> 14.3 mm
- net L_out: track 0.00 -> 13.5 mm
- net Net-(C8-Pad1): track 0.00 -> 12.5 mm
- net Net-(C9-Pad1): track 0.00 -> 5.01 mm
- net +9V: track 64.5 -> 63.6 mm
Other:
- board text added: "+"
- board text added: "L"
- board text added: "R"
